File: Hardware/BastWiFi.sch (KiCad schematic (older format))
At the start: 27 parts, among them J1 Conn_Battery, J3 Conn_Left, J4 Conn_Right, P1 USB_C_Plug_USB2.0, Q1 DMG3415U-7, SW1 GPIO0, SW2 RESET, U1 MCP73831-3-OT, U2 AP2112K-3.3, U3 ESP32-S2-WROVER

Commit message: Change footprint sw
Parts:
- SW1, SW2: footprint Button_Switch_SMD:SW_SPST_TL3342 -> Button_Switch_SMD:SW_SPST_B3U-1000P
Changed lines of the file:
@@
 F 0 "SW1" H 9390 5460 50  0000 C CNN
 F 1 "GPIO0" H 9390 5369 50  0000 C CNN
-F 2 "Button_Switch_SMD:SW_SPST_TL3342" H 9390 5375 50  0001 C CNN
+F 2 "Button_Switch_SMD:SW_SPST_B3U-1000P" H 9390 5375 50  0001 C CNN
 F 3 "~" H 9390 5375 50  0001 C CNN
 	1    9390 5175
@@
 F 0 "SW2" H 9390 6015 50  0000 C CNN
 F 1 "RESET" H 9390 5924 50  0000 C CNN
-F 2 "Button_Switch_SMD:SW_SPST_TL3342" H 9390 5930 50  0001 C CNN
+F 2 "Button_Switch_SMD:SW_SPST_B3U-1000P" H 9390 5930 50  0001 C CNN
 F 3 "~" H 9390 5930 50  0001 C CNN
 	1    9390 5730

Commit message: Add connector
Parts:
- P1: footprint (none) -> Connectors EC:C393939
Changed lines of the file:
@@
 F 0 "P1" H 7602 6262 50  0000 C CNN
 F 1 "USB_C_Plug_USB2.0" H 7602 6171 50  0000 C CNN
-F 2 "" H 7645 5395 50  0001 C CNN
+F 2 "Connectors EC:C393939" H 7645 5395 50  0001 C CNN
 F 3 "https://www.usb.org/sites/default/files/documents/usb_type-c.zip" H 7645 5395 50  0001 C CNN
 	1    7495 5395
