File: Hardware/BastWiFi.sch (KiCad schematic (older format))
At the start: 27 parts, among them J1 Conn_Battery, J3 Conn_Left, J4 Conn_Right, P1 USB_C_Plug_USB2.0, Q1 DMG3415U-7, SW1 GPIO0, SW2 RESET, U1 MCP73831-3-OT, U2 AP2112K-3.3, U3 ESP32-S2-WROVER

Commit message: Add button
Parts:
- SW1, SW2: footprint Button_Switch_SMD:SW_SPST_B3U-1000P -> Button_Switch_SMD:SW_SPST_PTS810
Changed lines of the file:
@@
 F 0 "SW1" H 9390 5460 50  0000 C CNN
 F 1 "GPIO0" H 9390 5369 50  0000 C CNN
-F 2 "Button_Switch_SMD:SW_SPST_B3U-1000P" H 9390 5375 50  0001 C CNN
+F 2 "Button_Switch_SMD:SW_SPST_PTS810" H 9390 5375 50  0001 C CNN
 F 3 "~" H 9390 5375 50  0001 C CNN
 	1    9390 5175
@@
 F 0 "SW2" H 9390 6015 50  0000 C CNN
 F 1 "RESET" H 9390 5924 50  0000 C CNN
-F 2 "Button_Switch_SMD:SW_SPST_B3U-1000P" H 9390 5930 50  0001 C CNN
+F 2 "Button_Switch_SMD:SW_SPST_PTS810" H 9390 5930 50  0001 C CNN
 F 3 "~" H 9390 5930 50  0001 C CNN
 	1    9390 5730

Commit message: Change sch
Parts:
- SW1, SW2: footprint Button_Switch_SMD:SW_SPST_PTS810 -> Connectors EC:C45281
Changed lines of the file:
@@
 F 0 "SW1" H 9390 5460 50  0000 C CNN
 F 1 "GPIO0" H 9390 5369 50  0000 C CNN
-F 2 "Button_Switch_SMD:SW_SPST_PTS810" H 9390 5375 50  0001 C CNN
+F 2 "Connectors EC:C45281" H 9390 5375 50  0001 C CNN
 F 3 "~" H 9390 5375 50  0001 C CNN
 	1    9390 5175
@@
 F 0 "SW2" H 9390 6015 50  0000 C CNN
 F 1 "RESET" H 9390 5924 50  0000 C CNN
-F 2 "Button_Switch_SMD:SW_SPST_PTS810" H 9390 5930 50  0001 C CNN
+F 2 "Connectors EC:C45281" H 9390 5930 50  0001 C CNN
 F 3 "~" H 9390 5930 50  0001 C CNN
 	1    9390 5730

Commit message: Change footprint
Parts:
- SW1, SW2: footprint Connectors EC:C45281 -> Connectors EC:C455281
Changed lines of the file:
@@
 F 0 "SW1" H 9390 5460 50  0000 C CNN
 F 1 "GPIO0" H 9390 5369 50  0000 C CNN
-F 2 "Connectors EC:C45281" H 9390 5375 50  0001 C CNN
+F 2 "Connectors EC:C455281" H 9390 5375 50  0001 C CNN
 F 3 "~" H 9390 5375 50  0001 C CNN
 	1    9390 5175
@@
 F 0 "SW2" H 9390 6015 50  0000 C CNN
 F 1 "RESET" H 9390 5924 50  0000 C CNN
-F 2 "Connectors EC:C45281" H 9390 5930 50  0001 C CNN
+F 2 "Connectors EC:C455281" H 9390 5930 50  0001 C CNN
 F 3 "~" H 9390 5930 50  0001 C CNN
 	1    9390 5730

Commit message: update V1.0
Parts:
- U3: symbol RF_Module:ESP32-S2-WROVER -> BastWiFi-rescue:ESP32-S2-WROVER-RF_Module
Other:
- moved on the sheet: C3
Changed lines of the file:
@@
 $EndComp
 $Comp
-L RF_Module:ESP32-S2-WROVER U3
+L BastWiFi-rescue:ESP32-S2-WROVER-RF_Module U3
 U 1 1 5EA53B09
 P 9425 2640
@@
 $EndComp
 Wire Wire Line
-	4720 3995 4725 3995
-Wire Wire Line
 	5650 3995 5650 3935
-Connection ~ 4725 3995
-Wire Wire Line
-	4725 3995 5430 3995
 $Comp
 L power:+BATT #PWR0129
@@
 L Device:C_Small C3
 U 1 1 5EAC5114
-P 5430 4095
-F 0 "C3" H 5522 4141 50  0000 L CNN
-F 1 "10uF" H 5522 4050 50  0000 L CNN
-F 2 "Capacitor_SMD:C_0603_1608Metric_Pad1.05x0.95mm_HandSolder" H 5430 4095 50  0001 C CNN
-F 3 "~" H 5430 4095 50  0001 C CNN
-	1    5430 4095
-	1    0    0    -1
-$EndComp
-Connection ~ 5430 3995
-Wire Wire Line
-	5430 3995 5650 3995
+P 5430 4160
+F 0 "C3" H 5522 4206 50  0000 L CNN
+F 1 "10uF" H 5522 4115 50  0000 L CNN
+F 2 "Capacitor_SMD:C_0603_1608Metric_Pad1.05x0.95mm_HandSolder" H 5430 4160 50  0001 C CNN
+F 3 "~" H 5430 4160 50  0001 C CNN
+	1    5430 4160
+	1    0    0    -1
+$EndComp
 $Comp
 L power:GND #PWR0130
 U 1 1 5EAC5C81
-P 5430 4195
-F 0 "#PWR0130" H 5430 3945 50  0001 C CNN
-F 1 "GND" H 5435 4022 50  0000 C CNN
-F 2 "" H 5430 4195 50  0001 C CNN
-F 3 "" H 5430 4195 50  0001 C CNN
-	1    5430 4195
+P 5430 4310
+F 0 "#PWR0130" H 5430 4060 50  0001 C CNN
+F 1 "GND" H 5435 4137 50  0000 C CNN
+F 2 "" H 5430 4310 50  0001 C CNN
+F 3 "" H 5430 4310 50  0001 C CNN
+	1    5430 4310
 	1    0    0    -1
 $EndComp
@@
 Text Label 980  2025 2    50   ~ 0
 A0
+Wire Wire Line
+	4725 3995 5430 3995
+Wire Wire Line
+	5430 4060 5430 3995
+Connection ~ 5430 3995
+Wire Wire Line
+	5430 3995 5650 3995
+Wire Wire Line
+	5430 4310 5430 4260
 $EndSCHEMATC
