File: Hardware/BastWiFi.sch (KiCad schematic (older format))
At the start: 27 parts, among them J1 Conn_Battery, J3 Conn_Left, J4 Conn_Right, P1 USB_C_Plug_USB2.0, Q1 DMG3415U-7, SW1 GPIO0, SW2 RESET, U1 MCP73831-3-OT, U2 AP2112K-3.3, U3 ESP32-S2-WROVER

Commit message: BOM
Parts:
- C1, C2, C3, C4, C5: manf# (none) -> CC0603KRX5R6BB106
- C6: manf# (none) -> 0603F104Z160CT
- C7: manf# (none) -> 885012106022
- D1: manf# (none) -> MBR120VLSFT3G
- P1: manf# (none) -> TYPE-C16PIN
- Q1: manf# (none) -> DMG3415U-7
- R1: manf# (none) -> CRCW06032K00FKEAC
- R2: manf# (none) -> RCA0603100KJNEC
- R3: manf# (none) -> ERJ-3GEYJ102V
- R4, R7, R8: manf# (none) -> SFR03EZPF1002
- R5, R6: manf# (none) -> CRCW06035K10FKEAC
- SW1, SW2: manf# (none) -> TS-1088R-02526
- U1: manf# (none) -> MCP73831T-2ACI/OT
- U2: manf# (none) -> AP2112K-3.3TRG1
- U3: manf# (none) -> ESP32-S2-WROVER
Changed lines of the file:
@@
 F 1 "ESP32-S2-WROVER" H 9875 3810 50  0000 C CNN
 F 2 "RF_Module:ESP32-S2-WROVER" H 10175 1490 50  0001 C CNN
-F 3 "https://www.espressif.com/sites/default/files/documentation/esp32-s2-wroom_esp32-s2-wroom-i_datasheet_en.pdf" H 9125 1840 50  0001 C CNN
+F 3 "https://www.mouser.mx/ProductDetail/Espressif-Systems/ESP32-S2-WROVER?qs=GBLSl2AkirtEnBxrL0jqTA%3D%3D" H 9125 1840 50  0001 C CNN
+F 4 "ESP32-S2-WROVER" H 9425 2640 50  0001 C CNN "manf#"
 	1    9425 2640
 	1    0    0    -1
@@
 F 1 "USB_C_Plug_USB2.0" H 7602 6171 50  0000 C CNN
 F 2 "Connectors EC:C393939" H 7645 5395 50  0001 C CNN
-F 3 "https://www.usb.org/sites/default/files/documents/usb_type-c.zip" H 7645 5395 50  0001 C CNN
+F 3 "https://lcsc.com/product-detail/USB-Connectors_SHOU-HAN-TYPE-C16PIN_C393939.html" H 7645 5395 50  0001 C CNN
+F 4 "TYPE-C16PIN" H 7495 5395 50  0001 C CNN "manf#"
 	1    7495 5395
 	1    0    0    -1
@@
 F 1 "AP2112K-3.3" H 5365 2290 50  0000 C CNN
 F 2 "Package_TO_SOT_SMD:SOT-23-5" H 5260 2375 50  0001 C CNN
-F 3 "https://www.diodes.com/assets/Datasheets/AP2112.pdf" H 5260 2150 50  0001 C CNN
+F 3 "https://www.mouser.mx/ProductDetail/Diodes-Incorporated/AP2112K-33TRG1?qs=%2Fha2pyFadugKN4ES11GMq2snst8wH3yje9KIABR%252BTfzTosnOVDqX4A%3D%3D" H 5260 2150 50  0001 C CNN
+F 4 "AP2112K-3.3TRG1" H 5260 2050 50  0001 C CNN "manf#"
 	1    5260 2050
 	1    0    0    -1
@@
 F 1 "MCP73831-3-OT" H 4705 4365 50  0000 C CNN
 F 2 "Package_TO_SOT_SMD:SOT-23-5" H 4375 3845 50  0001 L CIN
-F 3 "http://ww1.microchip.com/downloads/en/DeviceDoc/20001984g.pdf" H 4175 4045 50  0001 C CNN
+F 3 "https://www.mouser.mx/ProductDetail/Microchip-Technology/MCP73831T-2ACI-OT?qs=%2Fha2pyFadug7ns3NDcZ1%252BguMEttpm87FnqDgwUSDURWu9uo0PeBXyw%3D%3D" H 4175 4045 50  0001 C CNN
+F 4 "MCP73831T-2ACI/OT" H 4325 4095 50  0001 C CNN "manf#"
 	1    4325 4095
 	1    0    0    -1
@@
 F 1 "10uF" H 7545 1875 50  0000 L CNN
 F 2 "Capacitor_SMD:C_0603_1608Metric_Pad1.05x0.95mm_HandSolder" H 7695 1805 50  0001 C CNN
-F 3 "~" H 7695 1805 50  0001 C CNN
+F 3 "https://lcsc.com/product-detail/Others_YAGEO-CC0603KRX5R6BB106_C326057.html" H 7695 1805 50  0001 C CNN
+F 4 "CC0603KRX5R6BB106" H 7695 1805 50  0001 C CNN "manf#"
 	1    7695 1805
 	1    0    0    -1
@@
 F 1 "GPIO0" H 9390 5369 50  0000 C CNN
 F 2 "Connectors EC:C455281" H 9390 5375 50  0001 C CNN
-F 3 "~" H 9390 5375 50  0001 C CNN
+F 3 "https://lcsc.com/product-detail/New-Arrivals_XUNPU-TS-1088R-02526_C455281.html" H 9390 5375 50  0001 C CNN
+F 4 "TS-1088R-02526" H 9390 5175 50  0001 C CNN "manf#"
 	1    9390 5175
 	1    0    0    -1
@@
 F 1 "RESET" H 9390 5924 50  0000 C CNN
 F 2 "Connectors EC:C455281" H 9390 5930 50  0001 C CNN
-F 3 "~" H 9390 5930 50  0001 C CNN
+F 3 "https://lcsc.com/product-detail/New-Arrivals_XUNPU-TS-1088R-02526_C455281.html" H 9390 5930 50  0001 C CNN
+F 4 "TS-1088R-02526" H 9390 5730 50  0001 C CNN "manf#"
 	1    9390 5730
 	1    0    0    -1
@@
 F 1 "10K" H 10774 5305 50  0000 L CNN
 F 2 "Resistor_SMD:R_0603_1608Metric_Pad1.05x0.95mm_HandSolder" H 10715 5350 50  0001 C CNN
-F 3 "~" H 10715 5350 50  0001 C CNN
+F 3 "https://www.mouser.mx/ProductDetail/ROHM-Semiconductor/SFR03EZPF1002?qs=sGAEpiMZZMtlubZbdhIBIIR71ikvQRXL3s99k%2FjVgiA%3D" H 10715 5350 50  0001 C CNN
+F 4 "SFR03EZPF1002" H 10715 5350 50  0001 C CNN "manf#"
 	1    10715 5350
 	1    0    0    -1
@@
 F 1 "10K" H 10255 5315 50  0000 L CNN
 F 2 "Resistor_SMD:R_0603_1608Metric_Pad1.05x0.95mm_HandSolder" H 10440 5315 50  0001 C CNN
-F 3 "~" H 10440 5315 50  0001 C CNN
+F 3 "https://www.mouser.mx/ProductDetail/ROHM-Semiconductor/SFR03EZPF1002?qs=sGAEpiMZZMtlubZbdhIBIIR71ikvQRXL3s99k%2FjVgiA%3D" H 10440 5315 50  0001 C CNN
+F 4 "SFR03EZPF1002" H 10440 5315 50  0001 C CNN "manf#"
 	1    10440 5315
 	1    0    0    -1
@@
 F 1 "1uF" H 10807 5590 50  0000 L CNN
 F 2 "Capacitor_SMD:C_0603_1608Metric_Pad1.05x0.95mm_HandSolder" H 10715 5635 50  0001 C CNN
-F 3 "~" H 10715 5635 50  0001 C CNN
+F 3 "https://www.mouser.mx/ProductDetail/Wurth-Elektronik/885012106022?qs=%2Fha2pyFaduggjUC9vDyrNJ4O61U0x5QqpPCq9EfwtOf1CJEQO67jQw%3D%3D" H 10715 5635 50  0001 C CNN
+F 4 "885012106022" H 10715 5635 50  0001 C CNN "manf#"
 	1    10715 5635
 	1    0    0    -1
@@
 F 1 "0.1uF" H 7930 1745 50  0000 L CNN
 F 2 "Capacitor_SMD:C_0603_1608Metric_Pad1.05x0.95mm_HandSolder" H 7895 1805 50  0001 C CNN
-F 3 "~" H 7895 1805 50  0001 C CNN
+F 3 "https://lcsc.com/product-detail/Multilayer-Ceramic-Capacitors-MLCC-SMD-SMT_Walsin-Tech-Corp-0603F104Z160CT_C387984.html" H 7895 1805 50  0001 C CNN
+F 4 "0603F104Z160CT" H 7895 1805 50  0001 C CNN "manf#"
 	1    7895 1805
 	1    0    0    -1
@@
 F 1 "5.1K" V 8125 5140 50  0000 C CNN
 F 2 "Resistor_SMD:R_0603_1608Metric_Pad1.05x0.95mm_HandSolder" H 8195 4995 50  0001 C CNN
-F 3 "~" H 8195 4995 50  0001 C CNN
+F 3 "https://www.mouser.mx/ProductDetail/Vishay-Dale/CRCW06035K10FKEAC?qs=sGAEpiMZZMtlubZbdhIBIIZe04wfiaJW4mvAQUcl4N0%3D" H 8195 4995 50  0001 C CNN
+F 4 "CRCW06035K10FKEAC" V 8195 4995 50  0001 C CNN "manf#"
 	1    8195 4995
 	0    1    1    0
@@
 F 1 "5.1K" V 8265 5200 50  0000 C CNN
 F 2 "Resistor_SMD:R_0603_1608Metric_Pad1.05x0.95mm_HandSolder" H 8195 5095 50  0001 C CNN
-F 3 "~" H 8195 5095 50  0001 C CNN
+F 3 "https://www.mouser.mx/ProductDetail/Vishay-Dale/CRCW06035K10FKEAC?qs=sGAEpiMZZMtlubZbdhIBIIZe04wfiaJW4mvAQUcl4N0%3D" H 8195 5095 50  0001 C CNN
+F 4 "CRCW06035K10FKEAC" V 8195 5095 50  0001 C CNN "manf#"
 	1    8195 5095
 	0    1    1    0
@@
 F 1 "10uF" H 5812 2005 50  0000 L CNN
 F 2 "Capacitor_SMD:C_0603_1608Metric_Pad1.05x0.95mm_HandSolder" H 5720 2050 50  0001 C CNN
-F 3 "~" H 5720 2050 50  0001 C CNN
+F 3 "https://lcsc.com/product-detail/Others_YAGEO-CC0603KRX5R6BB106_C326057.html" H 5720 2050 50  0001 C CNN
+F 4 "CC0603KRX5R6BB106" H 5720 2050 50  0001 C CNN "manf#"
 	1    5720 2050
 	1    0    0    -1
@@
 F 1 "10uF" H 4465 2050 50  0000 L CNN
 F 2 "Capacitor_SMD:C_0603_1608Metric_Pad1.05x0.95mm_HandSolder" H 4700 2115 50  0001 C CNN
-F 3 "~" H 4700 2115 50  0001 C CNN
+F 3 "https://lcsc.com/product-detail/Others_YAGEO-CC0603KRX5R6BB106_C326057.html" H 4700 2115 50  0001 C CNN
+F 4 "CC0603KRX5R6BB106" H 4700 2115 50  0001 C CNN "manf#"
 	1    4700 2115
 	1    0    0    -1
@@
 F 1 "10K" H 4785 2115 50  0000 L CNN
 F 2 "Resistor_SMD:R_0603_1608Metric_Pad1.05x0.95mm_HandSolder" H 4960 2150 50  0001 C CNN
-F 3 "~" H 4960 2150 50  0001 C CNN
+F 3 "https://www.mouser.mx/ProductDetail/ROHM-Semiconductor/SFR03EZPF1002?qs=sGAEpiMZZMtlubZbdhIBIIR71ikvQRXL3s99k%2FjVgiA%3D" H 4960 2150 50  0001 C CNN
+F 4 "SFR03EZPF1002" H 4960 2150 50  0001 C CNN "manf#"
 	1    4960 2150
 	1    0    0    -1
@@
 F 1 "2K" H 3864 4290 50  0000 L CNN
 F 2 "Resistor_SMD:R_0603_1608Metric_Pad1.05x0.95mm_HandSolder" H 3805 4335 50  0001 C CNN
-F 3 "~" H 3805 4335 50  0001 C CNN
+F 3 "https://www.mouser.mx/ProductDetail/Vishay-Dale/CRCW06032K00FKEAC?qs=sGAEpiMZZMtlubZbdhIBIIZe04wfiaJWgXeS%2Fn31AeQ%3D" H 3805 4335 50  0001 C CNN
+F 4 "CRCW06032K00FKEAC" H 3805 4335 50  0001 C CNN "manf#"
 	1    3805 4335
 	1    0    0    -1
@@
 F 1 "1K" H 4919 4305 50  0000 L CNN
 F 2 "Resistor_SMD:R_0603_1608Metric_Pad1.05x0.95mm_HandSolder" H 4860 4350 50  0001 C CNN
-F 3 "~" H 4860 4350 50  0001 C CNN
+F 3 "https://www.mouser.mx/ProductDetail/Panasonic/ERJ-3GEYJ102V?qs=66DK8nO8gJBFiTsClorqsA%3D%3D" H 4860 4350 50  0001 C CNN
+F 4 "ERJ-3GEYJ102V" H 4860 4350 50  0001 C CNN "manf#"
 	1    4860 4350
 	1    0    0    -1
@@
 F 2 "Diode_SMD:D_0603_1608Metric_Pad1.05x0.95mm_HandSolder" H 4860 4600 50  0001 C CNN
 F 3 "~" H 4860 4600 50  0001 C CNN
+F 4 "" V 4860 4600 50  0001 C CNN "manf#"
 	1    4860 4600
 	0    -1   -1   0
@@
 F 1 "10uF" H 5522 4115 50  0000 L CNN
 F 2 "Capacitor_SMD:C_0603_1608Metric_Pad1.05x0.95mm_HandSolder" H 5430 4160 50  0001 C CNN
-F 3 "~" H 5430 4160 50  0001 C CNN
+F 3 "https://lcsc.com/product-detail/Others_YAGEO-CC0603KRX5R6BB106_C326057.html" H 5430 4160 50  0001 C CNN
+F 4 "CC0603KRX5R6BB106" H 5430 4160 50  0001 C CNN "manf#"
 	1    5430 4160
 	1    0    0    -1
@@
 F 1 "10uF" H 3315 4115 50  0000 L CNN
 F 2 "Capacitor_SMD:C_0603_1608Metric_Pad1.05x0.95mm_HandSolder" H 3265 4185 50  0001 C CNN
-F 3 "~" H 3265 4185 50  0001 C CNN
+F 3 "https://lcsc.com/product-detail/Others_YAGEO-CC0603KRX5R6BB106_C326057.html" H 3265 4185 50  0001 C CNN
+F 4 "CC0603KRX5R6BB106" H 3265 4185 50  0001 C CNN "manf#"
 	1    3265 4185
 	1    0    0    -1
@@
 F 1 "DMG3415U-7" H 4544 1705 50  0000 L CNN
 F 2 "Package_TO_SOT_SMD:TSOT-23" H 4540 1675 50  0001 L CIN
-F 3 "http://www.vishay.com/docs/70209/70209.pdf" H 4340 1750 50  0001 L CNN
+F 3 "https://www.mouser.mx/ProductDetail/Diodes-Incorporated/DMG3415U-7?qs=%2Fha2pyFaduj%252B8yiSwVhN6u3swdQLoENzjrkBSrNhwAg5xphgkJMLvw%3D%3D" H 4340 1750 50  0001 L CNN
+F 4 "DMG3415U-7" H 4340 1750 50  0001 C CNN "manf#"
 	1    4340 1750
 	1    0    0    -1
@@
 F 1 "MBR120" H 4235 2060 50  0000 C CNN
 F 2 "Diode_SMD:D_SOD-123F" H 4240 1775 50  0001 C CNN
-F 3 "http://www.onsemi.com/pub_link/Collateral/MBR340-D.PDF" H 4240 1950 50  0001 C CNN
+F 3 "https://www.mouser.mx/ProductDetail/ON-Semiconductor/MBR120VLSFT3G?qs=sGAEpiMZZMtQ8nqTKtFS%2FCKUxMvjsmGz%2FCigMfHc%252BQw%3D" H 4240 1950 50  0001 C CNN
+F 4 "MBR120VLSFT3G" H 4240 1950 50  0001 C CNN "manf#"
 	1    4240 1950
 	-1   0    0    1
@@
 F 1 "100K" H 3755 2040 50  0000 L CNN
 F 2 "Resistor_SMD:R_0603_1608Metric_Pad1.05x0.95mm_HandSolder" H 3995 2075 50  0001 C CNN
-F 3 "~" H 3995 2075 50  0001 C CNN
+F 3 "https://www.mouser.mx/ProductDetail/Vishay-Draloric/RCA0603100KJNEC?qs=DL%2Fp6SVo8Vmly4x%2FMjcyUQ==" H 3995 2075 50  0001 C CNN
+F 4 "RCA0603100KJNEC" H 3995 2075 50  0001 C CNN "manf#"
 	1    3995 2075
 	1    0    0    -1

Commit message: add LED
Parts:
- D2: manf# (none) -> 150060VS75000
Changed lines of the file:
@@
 F 1 "DONE" V 4808 4482 50  0000 R CNN
 F 2 "Diode_SMD:D_0603_1608Metric_Pad1.05x0.95mm_HandSolder" H 4860 4600 50  0001 C CNN
-F 3 "~" H 4860 4600 50  0001 C CNN
-F 4 "" V 4860 4600 50  0001 C CNN "manf#"
+F 3 "https://www.mouser.mx/ProductDetail/Wurth-Elektronik/150060VS75000?qs=LlUlMxKIyB1Q1Bi5mQ%2FKLw%3D%3D" H 4860 4600 50  0001 C CNN
+F 4 "150060VS75000" V 4860 4600 50  0001 C CNN "manf#"
 	1    4860 4600
 	0    -1   -1   0

Commit message: Add Connector
Parts:
- J1: manf# (none) -> B2B-PH-SM4-TB(LF)(SN)
Changed lines of the file:
@@
 F 1 "Conn_Battery" H 6425 4045 50  0000 C CNN
 F 2 "Connector_JST:JST_PH_B2B-PH-SM4-TB_1x02-1MP_P2.00mm_Vertical" H 6375 4145 50  0001 C CNN
-F 3 "~" H 6375 4145 50  0001 C CNN
+F 3 "https://lcsc.com/product-detail/Wire-To-Board-Wire-To-Wire-Connector_JST-Sales-America_B2B-PH-SM4-TB-LF-SN_JST-Sales-America-B2B-PH-SM4-TB-LF-SN_C160352.html" H 6375 4145 50  0001 C CNN
+F 4 "B2B-PH-SM4-TB(LF)(SN)" H 6375 4145 50  0001 C CNN "manf#"
 	1    6375 4145
 	0    -1   -1   0

Commit message: Add LED
Parts:
- added D3: LED, LED_SMD:LED_0603_1608Metric_Pad1.05x0.95mm_HandSolder, symbol Device:LED
- added R9: 1K, Resistor_SMD:R_0603_1608Metric_Pad1.05x0.95mm_HandSolder, symbol Device:R_Small
Connections:
- net GND: now also R9.2
- net GPIO13: now also D3.2 (A)
- new net: D3.1 (K), R9.1
Other:
- note added: "LED"
Changed lines of the file:
@@
 	2945 3245 6955 3245
-Wire Notes Line
-	6975 5320 2955 5320
 Wire Notes Line
 	2955 495  2955 5320
@@
 Wire Wire Line
 	5430 4310 5430 4260
+Wire Notes Line
+	480  5320 6975 5320
+$Comp
+L Device:LED D3
+U 1 1 5EFD0A27
+P 1655 3880
+F 0 "D3" H 1648 4097 50  0000 C CNN
+F 1 "LED" H 1648 4006 50  0000 C CNN
+F 2 "LED_SMD:LED_0603_1608Metric_Pad1.05x0.95mm_HandSolder" H 1655 3880 50  0001 C CNN
+F 3 "~" H 1655 3880 50  0001 C CNN
+	1    1655 3880
+	1    0    0    -1
+$EndComp
+$Comp
+L power:GND #PWR01
+U 1 1 5EFD13E3
+P 1290 4170
+F 0 "#PWR01" H 1290 3920 50  0001 C CNN
+F 1 "GND" H 1295 3997 50  0000 C CNN
+F 2 "" H 1290 4170 50  0001 C CNN
+F 3 "" H 1290 4170 50  0001 C CNN
+	1    1290 4170
+	1    0    0    -1
+$EndComp
+$Comp
+L Device:R_Small R9
+U 1 1 5EFD1BEC
+P 1290 4005
+F 0 "R9" H 1125 4045 50  0000 L CNN
+F 1 "1K" H 1120 3975 50  0000 L CNN
+F 2 "Resistor_SMD:R_0603_1608Metric_Pad1.05x0.95mm_HandSolder" H 1290 4005 50  0001 C CNN
+F 3 "https://www.mouser.mx/ProductDetail/Vishay-Dale/CRCW06032K00FKEAC?qs=sGAEpiMZZMtlubZbdhIBIIZe04wfiaJWgXeS%2Fn31AeQ%3D" H 1290 4005 50  0001 C CNN
+F 4 "CRCW06032K00FKEAC" H 1290 4005 50  0001 C CNN "manf#"
+	1    1290 4005
+	1    0    0    -1
+$EndComp
+Text Label 1805 3880 0    50   ~ 0
+GPIO13
+Wire Wire Line
+	1290 4105 1290 4170
+Wire Wire Line
+	1290 3880 1290 3905
+Text Notes 1215 3475 2    50   ~ 0
+LED
+Wire Wire Line
+	1290 3880 1505 3880
 $EndSCHEMATC
