File: Hardware/BastWiFi.kicad_pcb (KiCad board)
At the start: 2 copper layers, 60 x 22.9 mm, 37 parts, among them J1 Conn_Battery, J3 Conn_Left, J4 Conn_Right, P1 USB_C_Plug_USB2.0, Q1 DMG3415U-7, SW1 GPIO0, SW2 RESET, U1 MCP73831-3-OT, U2 AP2112K-3.3, U3 ESP32-S2-WROVER

Commit message: Change_name_pin
Other:
- board text added: "NC"
- board text removed: "MISC"
Changed lines of the file:
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@@
   (general
     (thickness 1.6)
-    (drawings 48)
+    (drawings 49)
     (tracks 507)
     (zones 0)
@@
       (rotate (xyz 0 0 180))
     )
+    (model "C:/Users/Diego Armadillo/Desktop/Documentos_EC/Modelos 3d/Bastwf/User Library-S2B-PH-SM4-TB.STEP"
+      (offset (xyz 0 5.5 0))
+      (scale (xyz 1 1 1))
+      (rotate (xyz 0 0 -180))
+    )
   )
   (module RF_Module:ESP32-S2-WROVER (layer F.Cu)
@@
       (rotate (xyz 0 0 0))
     )
+    (model "C:/Users/Diego Armadillo/Desktop/Documentos_EC/Modelos 3d/Bastwf/ESP32-S2-WROVER.STEP"
+      (offset (xyz 0 3.5 0))
+      (scale (xyz 1 1 1))
+      (rotate (xyz 0 0 0))
+    )
   )
   (module Package_TO_SOT_SMD:SOT-23-5 (layer F.Cu)
@@
       (rotate (xyz 0 0 0))
     )
+    (model "C:/Users/Diego Armadillo/Desktop/Documentos_EC/Modelos 3d/Bastwf/HRO_TYPE-C-31-M-12.step"
+      (offset (xyz -4.5 -7 0))
+      (scale (xyz 1 1 1))
+      (rotate (xyz 0 0 0))
+    )
   )
   (module "Connectors EC:C455281" (layer F.Cu)
@@
       (rotate (xyz -90 0 0))
     )
+    (model "C:/Users/Diego Armadillo/Desktop/Documentos_EC/Modelos 3d/Bastwf/3x4x2 tact button.step"
+      (offset (xyz 0 -0.5 0))
+      (scale (xyz 1 1 1))
+      (rotate (xyz -90 0 0))
+    )
   )
   (module "Connectors EC:C455281" (layer F.Cu)
@@
       (rotate (xyz -90 0 0))
     )
+    (model "C:/Users/Diego Armadillo/Desktop/Documentos_EC/Modelos 3d/Bastwf/3x4x2 tact button.step"
+      (offset (xyz 0 -0.5 0))
+      (scale (xyz 1 1 1))
+      (rotate (xyz -90 0 0))
+    )
   )
   (module LED_SMD:LED_0603_1608Metric_Pad1.05x0.95mm_HandSolder (layer F.Cu)
@@
     )
   )
+  (gr_text NC (at 138.38 100.49 90) (layer B.SilkS)
+    (effects (font (size 1 1) (thickness 0.15)) (justify mirror))
+  )
+  (gr_text NC (at 171.53 100.91 90) (layer B.SilkS)
+    (effects (font (size 1 1) (thickness 0.15)) (justify mirror))
+  )
   (gr_text Reset (at 137.2 98.1) (layer F.SilkS)
     (effects (font (size 0.8 0.8) (thickness 0.12)))
@@
     (effects (font (size 1 1) (thickness 0.15)))
   )
-  (gr_text MISC (at 171.5 100.06 90) (layer B.SilkS)
-    (effects (font (size 1 1) (thickness 0.15)) (justify mirror))
-  )
   (gr_text TX (at 168.87 100.7 90) (layer B.SilkS)
